File: pcb/mainboard/[DFR1142]Lite Carrier for LattePanda Mu.kicad_sch (KiCad schematic)
At the start: 6 parts

Commit message: before i aply ungrounding changes to moutning holes
Connections:
- removed net GND: H1.1, H2.1, H3.1, H4.1
