File: pcb/mainboard/[DFR1142]Lite Carrier for LattePanda Mu.kicad_pcb (KiCad board)
At the start: 4 copper layers, 115.5 x 127.2 mm, 166 parts, among them J1 Conn_01x03_Pin, J10 Conn_01x03_Pin, J11 Conn_01x03_Pin, J12 Conn_01x04_Pin, J13 Conn_01x04_Pin, J14 Conn_01x03_Pin, J15 Bus_M.2_Socket_M, J16 Bus_M.2_Socket_E, J3 HDMI_A, J7 Conn_01x04_Pin, J78 Conn_01x02_Pin, J79 USB3_A, J8 Conn_01x03_Pin, J80 USB3_A, J81 USB_C_Receptacle_USB2.0_16P, J82 Conn_01x04_Pin, J83 Conn_01x02_Pin, J9 Conn_01x04_Pin, Q1 2N7002, Q2 2SK3018, Q3 2SK3018, Q4 2SK3018, Q8 2N7002, U1 TPAZ1023-04F, U10 ULC0524P, U11 ULC0524P, U12 ULC0524P, U15 SY8253ADC, U16 SY8253ADC, U2 TPAZ1023-04F, U3 ULC0524P, U4 ULC0524P, U5 ULC0524P, U78 ULC0524P, U9 ULC0524P

Commit message: a lot more routing has been done now
Parts:
- removed BT1: Battery_Cell, A_HDJ_Library:Battery_Holder_CR1220_S8411-45R
- added H79: MountingHole_Pad, A_HDJ_Library:MountingHole_3mm_M2_Pad_TopOnly, F.Cu at (191.8, 73.5)
- added H80: MountingHole_Pad, A_HDJ_Library:MountingHole_3mm_M2_Pad_TopOnly, F.Cu at (128.2, 73.5)
- added J84: Conn_01x02_Pin, Connector_PinHeader_2.54mm:PinHeader_1x02_P2.54mm_Vertical, F.Cu at (152.8, 95.6)
- moved J78 260.3 mm to (195.8, 62.7)
- moved R76 251.5 mm to (175.2, 137.2), turned to -90 degrees
- moved R77 249.9 mm to (174.2, 137.2), turned to -90 degrees
- moved R2 237.8 mm to (159.6, 136.9), turned to -90 degrees
- moved Q1 236.7 mm to (181.9, 158.6)
- moved D4 236.3 mm to (181.1, 152.3), turned to 90 degrees
- moved D2 236.3 mm to (185.2, 159.6), turned to 180 degrees
- moved TP7 233.5 mm to (160.8, 139.2)
- moved R1 232.9 mm to (153.4, 136.8), turned to 180 degrees
- moved R6 231.5 mm to (184.8, 158.0), turned to -90 degrees
- moved R11 231.2 mm to (185.8, 158.0), turned to -90 degrees
- moved R4 228.2 mm to (179.2, 158.9), turned to -90 degrees
- moved D1 227.3 mm to (177.8, 152.3), turned to -90 degrees
- moved D3 226.8 mm to (177.8, 154.8), turned to -90 degrees
- moved Q2 226.5 mm to (175.1, 152.8)
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Routing:
- net /LattePanda Module/REFCLK3+: track 0.00 -> 59.4 mm
- net /LattePanda Module/REFCLK3-: track 0.00 -> 59.4 mm
- net /LattePanda Module/USB_2_P7+: track 0.00 -> 58.8 mm, vias 0 -> 2
- net /LattePanda Module/USB_2_P7-: track 0.00 -> 58.7 mm, vias 0 -> 2
- net /LattePanda Module/REFCLK0-: track 0.00 -> 50.1 mm, vias 0 -> 2
- net /LattePanda Module/REFCLK0+: track 0.00 -> 50.0 mm, vias 0 -> 2
- net /LattePanda Module/HSIO_2_RX-: track 28.6 -> 44.7 mm
- net /LattePanda Module/HSIO_2_RX+: track 28.7 -> 44.8 mm
- net /LattePanda Module/HSIO_3_RX+: track 45.9 -> 61.7 mm
- net /LattePanda Module/HSIO_3_RX-: track 46.0 -> 61.7 mm
- net /M.2 E&M Key/CON_PCIE_TX_1+: track 44.0 -> 43.1 mm
- net /M.2 E&M Key/CON_PCIE_TX_1-: track 44.1 -> 43.2 mm
- net GND: vias 0 -> 73

Commit message: components all now placed
Parts:
- removed H5, H6: MountingHole_Pad, A_HDJ_Library:MountingHole_3mm_M2_Pad_TopOnly
- moved TP4 279.2 mm to (197.8, 59.0)
- moved D17 274.6 mm to (189.6, 64.0), turned to 90 degrees
- moved D16 269.2 mm to (185.1, 64.0), turned to 90 degrees
- moved D15 263.9 mm to (180.5, 64.0), turned to 90 degrees
- moved TP13 256.6 mm to (166.5, 142.2)
- moved F1 242.3 mm to (188.8, 160.5), turned to 90 degrees
- moved D24 241.8 mm to (166.5, 139.1)
- moved R53 234.8 mm to (166.2, 137.2), turned to 180 degrees
- moved C25 227.7 mm to (187.5, 161.0), turned to 90 degrees
- moved R78 212.5 mm to (147.5, 100.5), turned to 90 degrees
- moved R79 210.4 mm to (145.8, 100.5), turned to 90 degrees
- moved R33 181.7 mm to (87.2, 140.5)
- moved R27 181.7 mm to (106.0, 120.5)
- moved FID1 179.2 mm to (185.8, 44.0)
- moved R32 173.2 mm to (99.8, 120.5)
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
Commit message: routing almost completely done if not done exept gnd
Parts:
- added FID1: Fiducial, A_HDJ_Library:Fiducial_0.5mm_Mask1mm, F.Cu at (129.5, 45.2)
- moved TP7 43.8 mm to (157.5, 137.8)
- moved R33 24.4 mm to (102.3, 121.2)
- moved FID2 12.9 mm to (120.8, 158.0)
- moved C32 5.23 mm to (90.5, 154.2)
- moved F5 5.23 mm to (93.2, 154.2)
- moved TP5 3.97 mm to (94.5, 107.2)
- moved C51 2.89 mm to (95.8, 142.8)
- moved C52 2.89 mm to (95.8, 141.8)
- moved C53 2.89 mm to (95.8, 144.8)
- moved C54 2.89 mm to (95.8, 143.8)
- moved R34 2.89 mm to (94.0, 141.3)
- moved R35 2.89 mm to (92.9, 141.3)
- moved TP6 2.87 mm to (95.2, 89.5)
- moved Q4 1.93 mm to (169.2, 147.2)
- moved R19 1.93 mm to (168.8, 144.7)
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Routing:
- net +3V3: track 0.00 -> 400.4 mm, vias 0 -> 9
- net VDC: track 0.00 -> 309.9 mm, vias 0 -> 32
- net +5V: track 0.00 -> 236.6 mm
- net /LattePanda Module/SLS_S3: track 0.00 -> 140.7 mm, vias 0 -> 4
- net /LattePanda Module/~{PWR_SW}: track 0.00 -> 100.2 mm, vias 0 -> 6
- net /~{PWR_LED}/~{PSON}: track 0.00 -> 99.0 mm, vias 0 -> 4
- net /GPIO/SOC_UART0_RX: track 0.00 -> 61.0 mm, vias 0 -> 2
- net /GPIO/SOC_UART1_RX: track 0.00 -> 58.7 mm, vias 0 -> 2
- net /GPIO/SOC_UART2_RX: track 0.00 -> 58.6 mm, vias 0 -> 2
- net /GPIO/SOC_UART0_TX: track 0.00 -> 51.4 mm, vias 0 -> 2
- net /GPIO/I2C2_SDA: track 0.00 -> 49.8 mm
- net /GPIO/SOC_UART1_TX: track 0.00 -> 46.7 mm, vias 0 -> 2
- net /GPIO/SOC_UART2_TX: track 0.00 -> 45.8 mm, vias 0 -> 2
- net /GPIO/I2C3_SDA: track 0.00 -> 45.2 mm
- net /GPIO/I2C4_SDA: track 0.00 -> 42.5 mm
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Other:
- board size 115.5 x 127.2 mm -> 116 x 127.2 mm
- board text added: "BAT"
- board text added: "DEBUG"
- board text added: "GND 3V3"
- board text added: "TX RX GND"

Commit message: before loading 12v in change
Routing:
- net +5V: track 236.6 -> 258.0 mm, vias 0 -> 2
- net +3V3: track 400.4 -> 407.0 mm
Changed lines of the file:
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@@
 	)
 	(segment
+		(start 176.8 160.05)
+		(end 178.5 161.75)
+		(width 0.4)
+		(layer "F.Cu")
+		(net 200)
+	)
+	(segment
 		(start 93 105.5)
 		(end 93 102.1)
@@
 	)
 	(segment
+		(start 171.375 160.05)
+		(end 176.8 160.05)
+		(width 0.4)
+		(layer "F.Cu")
+		(net 200)
+	)
+	(segment
 		(start 93 105.75)
 		(end 94.5 107.25)
@@
 	)
 	(segment
+		(start 179.75 161.75)
+		(end 180.5 161)
+		(width 0.4)
+		(layer "F.Cu")
+		(net 200)
+	)
+	(segment
 		(start 89.01 104.05)
 		(end 89.01 103.93)
@@
 	)
 	(segment
+		(start 181.05 151.25)
+		(end 181.1 151.3)
+		(width 0.4)
+		(layer "F.Cu")
+		(net 200)
+	)
+	(segment
 		(start 89.03 105.1)
 		(end 89.03 106.495)
@@
 	)
 	(segment
+		(start 180 151.25)
+		(end 181.05 151.25)
+		(width 0.4)
+		(layer "F.Cu")
+		(net 200)
+	)
+	(segment
 		(start 88.775 109.985)
 		(end 88.76 109.97)
@@
 	)
 	(segment
+		(start 178.5 161.75)
+		(end 179.75 161.75)
+		(width 0.4)
+		(layer "F.Cu")
+		(net 200)
+	)
+	(segment
 		(start 89 118.75)
 		(end 89 135.25)
@@
 		(net 200)
 	)
+	(via
+		(at 180 151.25)
+		(size 0.4)
+		(drill 0.2)
+		(layers "F.Cu" "B.Cu")
+		(net 200)
+	)
+	(via
+		(at 180.5 161)
+		(size 0.4)
+		(drill 0.2)
+		(layers "F.Cu" "B.Cu")
+		(net 200)
+	)
+	(segment
+		(start 180.5 161)
+		(end 180.5 157.25)
+		(width 0.4)
+		(layer "In2.Cu")
+		(net 200)
+	)
+	(segment
+		(start 179.75 156.5)
+		(end 179.75 151.5)
+		(width 0.4)
+		(layer "In2.Cu")
+		(net 200)
+	)
+	(segment
+		(start 180.5 157.25)
+		(end 179.75 156.5)
+		(width 0.4)
+		(layer "In2.Cu")
+		(net 200)
+	)
+	(segment
+		(start 179.75 151.5)
+		(end 180 151.25)
+		(width 0.4)
+		(layer "In2.Cu")
+		(net 200)
+	)
 	(segment
 		(start 132 139)
@@
 	)
 	(segment
+		(start 174.2125 155.3375)
+		(end 174.2125 155.858032)
+		(width 0.2)
+		(layer "F.Cu")
+		(net 203)
+	)
+	(segment
 		(start 89.675 90.4)
 		(end 89.675 88.815)
@@
 	)
 	(segment
+		(start 174.2125 155.858032)
+		(end 176.734468 158.38)
+		(width 0.2)
+		(layer "F.Cu")
+		(net 203)
+	)
+	(segment
 		(start 172.2 154.96)
 		(end 173.835 154.96)
@@
 	)
 	(segment
+		(start 176.734468 158.38)
+		(end 179.25 158.38)
+		(width 0.2)
+		(layer "F.Cu")
+		(net 203)
+	)
+	(segment
 		(start 84.651 77.5)
 		(end 84.651 97.249)
@@
 	)
 	(zone
+		(net 203)
+		(net_name "+3V3")
+		(layer "F.Cu")
+		(name "$teardrop_padvia$")
+		(hatch none 0.1)
+		(priority 30000)
+		(attr
+			(teardrop
+				(type padvia)
+			)
+		)
+		(connect_pads yes
+			(clearance 0)
+		)
+		(min_thickness 0.0254)
+		(filled_areas_thickness no)
+		(fill yes
+			(thermal_gap 0.5)
+			(thermal_bridge_width 0.5)
+			(island_removal_mode 1)
+			(island_area_min 10)
+		)
+		(polygon
+			(pts
+				(xy 174.339403 155.843514) (xy 174.345024 155.770093) (xy 174.363321 155.729434) (xy 174.393253 155.691932)
+				(xy 174.428541 155.665492) (xy 174.473455 155.646649) (xy 174.542878 155.6375) (xy 174.211793 155.336793)
+				(xy 173.939972 155.6375) (xy 174.004723 155.655771) (xy 174.071247 155.713917) (xy 174.139347 155.821321)
+				(xy 174.193348 155.964791) (xy 174.197982 155.984935)
+			)
+		)
+	)
+	(zone
 		(net 220)
 		(net_name "Net-(D22-K)")
@@
 	)
 	(zone
+		(net 200)
+		(net_name "+5V")
+		(layer "F.Cu")
+		(name "$teardrop_padvia$")
+		(hatch none 0.1)
+		(priority 30000)
+		(attr
+			(teardrop
+				(type padvia)
+			)
+		)
+		(connect_pads yes
+			(clearance 0)
+		)
+		(min_thickness 0.0254)
+		(filled_areas_thickness no)
+		(fill yes
+			(thermal_gap 0.5)
+			(thermal_bridge_width 0.5)
+			(island_removal_mode 1)
+			(island_area_min 10)
+		)
+		(polygon
+			(pts
+				(xy 172.275 159.85) (xy 172.121856 159.841988) (xy 172.031296 159.828583) (xy 171.939875 159.805901)
+				(xy 171.863006 159.776116) (xy 171.794941 159.735623) (xy 171.752364 159.697282) (xy 171.719127 159.651359)
+				(xy 171.697887 159.6) (xy 171.374 160.05) (xy 171.697887 160.5) (xy 171.740787 160.416348) (xy 171.817379 160.348954)
+				(xy 171.933533 160.296116) (xy 172.093911 160.261357) (xy 172.275 160.25)
+			)
+		)
+	)
+	(zone
 		(net 315)
 		(net_name "/PSU/PWR_EN")
@@
 			)
 		)
+	)
+	(zone
+		(net 203)
+		(net_name "+3V3")
+		(layer "F.Cu")
+		(name "$teardrop_padvia$")
+		(hatch none 0.1)
+		(priority 30001)
+		(attr
+			(teardrop
+				(type padvia)
+			)
+		)
+		(connect_pads yes
+			(clearance 0)
+		)
+		(min_thickness 0.0254)
+		(filled_areas_thickness no)
+		(fill yes
+			(thermal_gap 0.5)
+			(thermal_bridge_width 0.5)
+			(island_removal_mode 1)
+			(island_area_min 10)
+		)
+		(polygon
+			(pts
+				(xy 178.66 158.48) (xy 178.744592 158.485925) (xy 178.845619 158.507398) (xy 178.911293 158.533373)
+				(xy 178.966987 158.570584) (xy 178.994863 158.602099) (xy 179.013338 158.639724) (xy 179.251 158.38)
+				(xy 179.013338 158.120276) (xy 178.974359 158.182452) (xy 178.899476 158.232326) (xy 178.783272 158.267862)
+				(xy 178.66 158.28)
+			)
+		)

Commit message: before i aply ungrounding changes to moutning holes
Parts:
- added J85: Conn_01x01_Pin, Connector_Wire:SolderWire-1sqmm_1x01_D1.4mm_OD2.7mm, F.Cu at (196.2, 54.5)
- J78: value Conn_01x02_Pin -> Conn_01x01_Pin; footprint Connector_PinHeader_2.54mm:PinHeader_1x02_P2.54mm_Vertical -> Connector_Wire:SolderWire-1sqmm_1x01_D1.4mm_OD2.7mm
- moved TP4 8.59 mm to (196.5, 67.5)
- moved TP5 7.00 mm to (101.5, 107.4)
- moved TP6 3.50 mm to (95.3, 93.0)
- moved J78 1.12 mm to (196.2, 63.8)
Routing:
- net +3V3: track 407.0 -> 488.8 mm, vias 9 -> 13
- net /LattePanda Module/SUSCLK_WIFI: track 1.21 -> 74.6 mm, vias 0 -> 6
- net /~{PLT_RST}: track 29.1 -> 97.0 mm, vias 4 -> 9
- net /~{WAKE}: track 22.1 -> 85.8 mm, vias 2 -> 6
- net GND: track 3.05 -> 45.4 mm
- net VDC: track 309.9 -> 341.6 mm, vias 32 -> 34
- net +5V: track 258.0 -> 265.0 mm
- net +12V: track 20.1 -> 16.5 mm
- net Net-(A1-TCP1_HPD): track 0.00 -> 2.27 mm
- net Net-(A1-TCP0_HPD): track 0.00 -> 2.12 mm
- net Net-(D9-A): track 0.00 -> 1.76 mm
Other:
- board text added: "12v"

Commit message: looking good i think done exept 23d models
Connections:
- H1 pad 1: GND -> unconnected-(H1-Pad1)
- H2 pad 1: GND -> unconnected-(H2-Pad1)
- H3 pad 1: GND -> unconnected-(H3-Pad1)
- H4 pad 1: GND -> unconnected-(H4-Pad1)
Routing:
- net GND: track 45.4 -> 400.0 mm, vias 73 -> 386
- net /~{PWR_LED}/~{PSON}: track 99.0 -> 204.6 mm, vias 4 -> 9
- added copper zone on B.Cu, net GND
- added copper zone on F.Cu, net GND
- added copper zone on In1.Cu, net GND
