File: pcb/mainboard/[DFR1142]Lite Carrier for LattePanda Mu.kicad_pcb (KiCad board)
At the start: 4 copper layers, 116 x 127.2 mm, 168 parts, among them J1 Conn_01x03_Pin, J10 Conn_01x03_Pin, J11 Conn_01x03_Pin, J12 Conn_01x04_Pin, J13 Conn_01x04_Pin, J14 Conn_01x03_Pin, J15 Bus_M.2_Socket_M, J16 Bus_M.2_Socket_E, J3 HDMI_A, J7 Conn_01x04_Pin, J78 Conn_01x01_Pin, J79 USB3_A, J8 Conn_01x03_Pin, J80 USB3_A, J81 USB_C_Receptacle_USB2.0_16P, J82 Conn_01x04_Pin, J83 Conn_01x02_Pin, J84 Conn_01x02_Pin, J85 Conn_01x01_Pin, J9 Conn_01x04_Pin, Q1 2N7002, Q2 2SK3018, Q3 2SK3018, Q4 2SK3018, Q8 2N7002, U1 TPAZ1023-04F, U10 ULC0524P, U11 ULC0524P, U12 ULC0524P, U15 SY8253ADC, U16 SY8253ADC, U2 TPAZ1023-04F, U3 ULC0524P, U4 ULC0524P, U5 ULC0524P, U78 ULC0524P, U9 ULC0524P

Commit message: pcb is ready for production
Routing:
- net /LattePanda Module/HSIO_2_RX+: track 44.8 -> 46.9 mm
- net /USB2.0&USB3.0/CON_USB3_D_N: track 25.8 -> 24.8 mm
- net /M.2 E&M Key/CON_PCIE_TX_0+: track 11.6 -> 12.5 mm
- net /LattePanda Module/HSIO_2_RX-: track 44.7 -> 45.5 mm
- net GND: track 400.0 -> 400.4 mm, vias 386 -> 391

Commit message: gerbers are ready all done
Other:
- board text added: "NOMAD V1"
