File: pcb/mainboard/[DFR1142]Lite Carrier for LattePanda Mu.kicad_pcb (KiCad board)
At the start: 4 copper layers, 116 x 127.2 mm, 168 parts, among them J1 Conn_01x03_Pin, J10 Conn_01x03_Pin, J11 Conn_01x03_Pin, J12 Conn_01x04_Pin, J13 Conn_01x04_Pin, J14 Conn_01x03_Pin, J15 Bus_M.2_Socket_M, J16 Bus_M.2_Socket_E, J3 HDMI_A, J7 Conn_01x04_Pin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

Commit message: updated
Other:
- board text added: "ADD GND PLANE TO L3"
