File: pcb/mainboard/USB2.0&USB3.0.kicad_sch (KiCad schematic)
At the start: 26 parts, among them J79 USB3_A, J80 USB3_A, J81 USB_C_Receptacle_USB2.0_16P, J82 Conn_01x04_Pin, U3 ULC0524P, U4 ULC0524P, U5 ULC0524P, U78 ULC0524P

Commit message: 510
Connections:
- net GND: now also U78.3 (VSS), U78.8 (VSS)
Other:
- note added: "but before there was no gnd"
- note added: "should be fine"
Changed lines of the file:
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@@
 		(company "DFRobot")
+	)
+	(text "but before there was no gnd"
+		(exclude_from_sim no)
+		(at 233.68 180.086 0)
+		(effects
+			(font
+				(size 1.27 1.27)
+			)
+		)
 	)
 	(text "usb 3 seperated\n"
@@
 		(exclude_from_sim no)
 		(at 313.69 143.764 0)
+		(effects
+			(font
+				(size 1.27 1.27)
+			)
+		)
+	)
+	(text "should be fine"
+		(exclude_from_sim no)
+		(at 232.41 178.308 0)
 		(effects
 			(font
@@
 					(unit 1)
 				)
+			)
+		)
+	)
+	(symbol
+		(lib_id "power:GND")
+		(at 232.41 173.99 270)
+		(unit 1)
+		(exclude_from_sim no)
+		(in_bom yes)
+		(on_board yes)
+		(dnp no)
+		(fields_autoplaced yes)
+		(property "Reference" "#PWR0122"
+			(at 226.06 173.99 0)
+			(effects
+				(font
+					(size 1.27 1.27)
+				)
+				(hide yes)
+			)
+		)
+		(property "Value" "GND"
+			(at 228.6 173.99 90)
+			(effects
+				(font
+					(size 1.27 1.27)
+				)
+				(justify right)
+			)
+		)
+		(property "Footprint" ""
+			(at 232.41 173.99 0)
+			(effects
+				(font
+					(size 1.27 1.27)
+				)
+				(hide yes)
+			)
+		)
+		(property "Datasheet" ""
+			(at 232.41 173.99 0)
+			(effects
+				(font
+					(size 1.27 1.27)
+				)
+				(hide yes)
+			)
+		)
+		(property "Description" ""
+			(at 232.41 173.99 0)
+			(effects
+				(font
+					(size 1.27 1.27)
+				)
+				(hide yes)
+			)
+		)
+		(pin "1"
+		)
+		(instances
+			(project "[DFR1142]Lite Carrier for LattePanda Mu"
+				(path "/2a6d114a-7fd7-4207-b5f7-4ea9c34f36aa/f9aa04f2-8362-4e9f-9e54-e2b1a8ec9b0a"
+					(reference "#PWR0122")
+					(unit 1)
+				)
