File: pcb V2/[DFR1142]Lite Carrier for LattePanda Mu.kicad_sch (KiCad schematic)
At the start: 6 parts

Commit message: 510
Parts:
- added A78: LattePanda_Mu, Module_LattePanda:LattePanda_Module_H8.0mm_Horizontal, symbol MCU_Module_LattePanda:LattePanda_Mu
- added C17, C18, C19, C20, C21, C22, C23, C24, C25, C26, C27, C28, C29: 100nF/50V, A_HDJ_Library:C_0402_1005Metric, symbol Device:C
- added C30, C31, C32, C86: 22uF/10V, A_HDJ_Library:C_0603_1608Metric, symbol Device:C
- added D1, D2, D3, D78, D79, D8, D80: ESD5V0B03, A_HDJ_Library:D_0402_1005Metric, symbol Diode:ESD9B5.0ST5G
- added D4: 1N5819WS, A_HDJ_Library:D_SOD-323, symbol Diode:1N5819WS
- added F1: 6V/50mA, A_HDJ_Library:R_0603_1608Metric, symbol Device:Fuse
- added F2, F78: 6V/1A, A_HDJ_Library:Fuse_0805_2012Metric, symbol Device:Fuse
- added F4: 6V/2A, A_HDJ_Library:R_0805_2012Metric, symbol Device:Fuse
- added F5: 6V/2A, A_HDJ_Library:Fuse_0805_2012Metric, symbol Device:Fuse
- added J1, J10, J11, J14, J8: Conn_01x03_Pin, A_HDJ_Library:PinHeader_1x03_P2.54mm_Vertical, symbol Connector:Conn_01x03_Pin
- added J12, J13, J7, J9: Conn_01x04_Pin, A_HDJ_Library:PinHeader_1x04_P2.54mm_Vertical, symbol Connector:Conn_01x04_Pin
- added J3: HDMI_A, A_HDJ_Library:HDMI_A_Molex_208658-1001_Horizontal, symbol Connector:HDMI_A
- added J79, J80: USB3_A, Connector_USB:USB3_A_Molex_48393-001, symbol Connector:USB3_A
- added J81: USB_C_Receptacle_USB2.0_16P, Connector_USB:USB_C_Receptacle_GCT_USB4085, symbol Connector:USB_C_Receptacle_USB2.0_16P
- added J82: Conn_01x04_Pin, Connector_PinHeader_2.54mm:PinHeader_1x04_P2.54mm_Vertical, symbol Connector:Conn_01x04_Pin
- added J84: Conn_01x02_Pin, Connector_PinHeader_2.54mm:PinHeader_1x02_P2.54mm_Vertical, symbol Connector:Conn_01x02_Pin
- added Q1: 2N7002, A_HDJ_Library:SOT-23, symbol Transistor_FET:2N7002
- added Q2, Q3, Q4: 2SK3018, A_HDJ_Library:SOT-23, symbol Transistor_FET:2N7002
- added R1, R11: 1K/1%, A_HDJ_Library:R_0402_1005Metric, symbol Device:R
- added R10, R13, R14, R16, R17, R7, R8, R9: 470R/1%, A_HDJ_Library:R_0402_1005Metric, symbol Device:R
- added R15, R18, R19, R3, R5: 2.2K/1%, A_HDJ_Library:R_0402_1005Metric, symbol Device:R
- added R2: 10K/1%, A_HDJ_Library:R_0402_1005Metric, symbol Device:R
- added R4: 1M/1%, A_HDJ_Library:R_0402_1005Metric, symbol Device:R
- added R6: 21.5K/1%, A_HDJ_Library:R_0402_1005Metric, symbol Device:R
- added R76, R77: 100K/1%, A_HDJ_Library:R_0402_1005Metric, symbol Device:R
- added R78, R79: 10K/1%, Resistor_SMD:R_0402_1005Metric, symbol Device:R
- added R80, R81: 5.1K/1%, A_HDJ_Library:R_0402_1005Metric, symbol Device:R
- added TP7: TestPoint, A_HDJ_Library:TestPoint_Pad_D1.5mm, symbol Connector:TestPoint
- added U1, U2: TPAZ1023-04F, A_HDJ_Library:Diodes_UDFN-10_1.0x2.5mm_P0.5mm, symbol Power_Protection:D3V3XA4B10LP
- added U10, U11, U12, U3, U4, U5, U78, U9: ULC0524P, A_HDJ_Library:Diodes_UDFN-10_1.0x2.5mm_P0.5mm, symbol Power_Protection:D3V3XA4B10LP
Connections:
- net ~{PLT_RST}: now also A78.105 (~{PLTRST})
- net ~{PWR_LED}/~{PSON}: now also A78.5 (SLS_S0), R19.1
- new net: F2.2, J81.A4 (VBUS), J81.A9 (VBUS), J81.B4 (VBUS), J81.B9 (VBUS), R80.1, R81.1
- new net: Q4.3 (D), R10.1, R13.1, R14.1, R16.1, R17.1, R7.1, R8.1, R9.1
- new net: J81.B5 (CC2), R81.2
- new net: U4.4, U4.7 (NC)
- new net: U4.5, U4.6 (NC)
- new net: F1.2, J3.18 (+5V)
- new net: F4.2, J79.1 (VBUS)
- new net: J84.2 (Pin_2), R1.2
- new net: Q1.3 (D), R11.1, R6.1
- new net: F78.2, J82.1 (Pin_1)
- new net: J81.A5 (CC1), R80.2
- new net: A78.187 (TCP0_HPD), R76.1
- new net: A78.100 (~{CLKREQ3}), R79.1
- new net: A78.102 (~{CLKREQ4}), R78.1
- new net: A78.185 (TCP1_HPD), R77.1
- new net: A78.133 (~{BIOS_SEL}), R2.1, TP7.1
- new net: A78.10 (SIO_UART_TX), J1.1 (Pin_1)
- new net: A78.12 (SIO_UART_RX), J1.2 (Pin_2)
- new net: Q4.1 (G), R19.2
- new net: F5.2, J80.1 (VBUS)
- new net: U10.5, U10.6 (NC)
- new net: U12.5, U12.6 (NC)
- new net +3V3: J13.1 (Pin_1), J13.2 (Pin_2), J13.3 (Pin_3), J13.4 (Pin_4), J14.1 (Pin_1), J14.2 (Pin_2), J14.3 (Pin_3), Q1.1 (G), Q2.1 (G), Q3.1 (G), R3.1, R4.1, R5.1
- new net +5V: C30.2, C31.2, C32.2, C86.2, D4.2 (A), F2.1, F4.1, F5.1, F78.1
- new net +BATT: A78.115 (VBAT), R1.1
- new net 5V_HDMI_VCC: C25.1, D4.1 (K), F1.1, R15.1, R18.1
- new net CON_USB3_SSTX_N: C26.2, J79.8 (SSTX-), U3.4, U3.7 (NC)
- new net CON_USB3_SSTX_P: C27.2, J79.9 (SSTX+), U3.5, U3.6 (NC)
- new net CON_USB4_SSTX_N: C28.2, J80.8 (SSTX-), U5.4, U5.7 (NC)
- new net CON_USB4_SSTX_P: C29.2, J80.9 (SSTX+), U5.5, U5.6 (NC)
- new net DDC_SCL: D1.2 (A2), J3.15 (SCL), Q2.3 (D), R15.2
- new net DDC_SDA: D3.2 (A2), J3.16 (SDA), Q3.3 (D), R18.2
- new net DDI_B_DDC_SCL: A78.171 (DDIB_DDC_SCL), Q2.2 (S), R5.2
- new net DDI_B_DDC_SDA: A78.169 (DDIB_DDC_SDA), Q3.2 (S), R3.2
- new net DDI_B_HPD: A78.183 (DDIB_HPD), Q1.2 (S), R4.2
- new net DDI_B_TX0+: A78.217 (DDIB_TX0+), C17.1
- new net DDI_B_TX0-: A78.215 (DDIB_TX0-), C18.1
- new net DDI_B_TX1+: A78.211 (DDIB_TX1+), C19.1
- new net DDI_B_TX1-: A78.209 (DDIB_TX1-), C20.1
- new net DDI_B_TX2+: A78.205 (DDIB_TX2+), C21.1
- new net DDI_B_TX2-: A78.203 (DDIB_TX2-), C22.1
- new net DDI_B_TX3+: A78.199 (DDIB_TX3+), C23.1
- new net DDI_B_TX3-: A78.197 (DDIB_TX3-), C24.1
- new net GND: A78.101 (GND), A78.107 (GND), A78.11 (GND), A78.110 (GND), A78.113 (GND), A78.116 (GND), A78.135 (GND), A78.136 (GND), A78.14 (GND), A78.151 (GND), A78.158 (GND), A78.167 (GND), A78.17 (GND), A78.170 (GND), A78.181 (GND), A78.182 (GND), A78.188 (GND), A78.189 (GND), A78.194 (GND), A78.195 (GND), A78.20 (GND), A78.200 (GND), A78.201 (GND), A78.206 (GND), A78.207 (GND), A78.212 (GND), A78.213 (GND), A78.218 (GND), A78.219 (GND), A78.224 (GND), A78.225 (GND), A78.23 (GND), A78.230 (GND), A78.231 (GND), A78.236 (GND), A78.237 (GND), A78.242 (GND), A78.243 (GND), A78.248 (GND), A78.249 (GND), A78.26 (GND), A78.29 (GND), A78.32 (GND), A78.35 (GND), A78.38 (GND), A78.41 (GND), A78.44 (GND), A78.47 (GND), A78.50 (GND), A78.53 (GND), A78.56 (GND), A78.59 (GND), A78.62 (GND), A78.65 (GND), A78.68 (GND), A78.71 (GND), A78.74 (GND), A78.77 (GND), A78.80 (GND), A78.83 (GND), A78.86 (GND), A78.89 (GND), A78.92 (GND), A78.95 (GND), A78.98 (GND), A78.MP (Mountinge_Pads), C25.2, C30.1, C31.1, C32.1, C86.1, D1.1 (A1), D2.1 (A1), D3.1 (A1), D78.1 (A1), D79.1 (A1), D8.1 (A1), D80.1 (A1), J1.3 (Pin_3), J11.1 (Pin_1), J11.2 (Pin_2), J11.3 (Pin_3), J12.1 (Pin_1), J12.2 (Pin_2), J12.3 (Pin_3), J12.4 (Pin_4), J3.11 (CKS), J3.17 (GND), J3.2 (D2S), J3.5 (D1S), J3.8 (D0S), J3.SH, J79.10 (SHIELD), J79.4 (GND), J79.7 (DRAIN), J80.10 (SHIELD), J80.4 (GND), J80.7 (DRAIN), J81.A1 (GND), J81.A12 (GND), J81.B1 (GND), J81.B12 (GND), J81.S1 (SHIELD), J82.4 (Pin_4), J84.1 (Pin_1), Q4.2 (S), R6.2, R76.2, R77.2, R78.2, R79.2, U1.3 (VSS), U1.8 (VSS), U10.3 (VSS), U10.8 (VSS), U11.3 (VSS), U11.8 (VSS), U12.3 (VSS), U12.8 (VSS), U2.3 (VSS), U2.8 (VSS), U3.3 (VSS), U3.8 (VSS), U4.3 (VSS), U4.8 (VSS), U5.3 (VSS), U5.8 (VSS), U78.3 (VSS), U78.8 (VSS), U9.3 (VSS), U9.8 (VSS)
- new net HPD: D2.2 (A2), J3.19 (HPD), R11.2
- new net HSIO_0_RX+: A78.16 (HSIO0_RX+)
- new net HSIO_0_RX-: A78.18 (HSIO0_RX-)
- new net HSIO_0_TX+: A78.13 (HSIO0_TX+)
- new net HSIO_0_TX-: A78.15 (HSIO0_TX-)
- new net HSIO_1_RX+: A78.22 (HSIO1_RX+)
- new net HSIO_1_RX-: A78.24 (HSIO1_RX-)
- new net HSIO_1_TX+: A78.19 (HSIO1_TX+)
- new net HSIO_1_TX-: A78.21 (HSIO1_TX-)
- new net HSIO_2_RX+: A78.28 (HSIO2_RX+)
- new net HSIO_2_RX-: A78.30 (HSIO2_RX-)
- new net HSIO_2_TX+: A78.25 (HSIO2_TX+)
- new net HSIO_2_TX-: A78.27 (HSIO2_TX-)
- new net HSIO_3_RX+: A78.34 (HSIO3_RX+)
- new net HSIO_3_RX-: A78.36 (HSIO3_RX-)
- new net HSIO_3_TX+: A78.31 (HSIO3_TX+)
- new net HSIO_3_TX-: A78.33 (HSIO3_TX-)
- new net HSIO_6_RX+: A78.64 (HSIO6_RX+)
- new net HSIO_6_RX-: A78.66 (HSIO6_RX-)
- new net HSIO_6_TX+: A78.61 (HSIO6_TX+)
- new net HSIO_6_TX-: A78.63 (HSIO6_TX-)
- new net I2C2_SCL: A78.154 (I2C2_SCL), J9.1 (Pin_1), U11.1, U11.10 (NC)
- new net I2C2_SDA: A78.156 (I2C2_SDA), J7.1 (Pin_1), U9.1, U9.10 (NC)
- new net I2C3_SCL: A78.150 (I2C3_SCL), J9.2 (Pin_2), U11.2, U11.9 (NC)
- new net I2C3_SDA: A78.152 (I2C3_SDA), J7.2 (Pin_2), U9.2, U9.9 (NC)
- new net I2C4_SCL: A78.146 (I2C4_SCL), J9.3 (Pin_3), U11.4, U11.7 (NC)
- new net I2C4_SDA: A78.148 (I2C4_SDA), J7.3 (Pin_3), U9.4, U9.7 (NC)
- new net I2C5_SCL: A78.142 (I2C5_SCL), J9.4 (Pin_4), U11.5, U11.6 (NC)
- new net I2C5_SDA: A78.144 (I2C5_SDA), J7.4 (Pin_4), U9.5, U9.6 (NC)
- new net REFCLK0+: A78.85 (REFCLK0+)
- new net REFCLK0-: A78.87 (REFCLK0-)
- new net REFCLK2+: A78.97 (REFCLK2+)
- new net REFCLK2-: A78.99 (REFCLK2-)
- new net REFCLK3+: A78.88 (REFCLK3+)
- new net REFCLK3-: A78.90 (REFCLK3-)
- new net REFCLK4+: A78.94 (REFCLK4+)
- new net REFCLK4-: A78.96 (REFCLK4-)
- new net SLS_S3: A78.7 (SLS_S3)
- new net SOC_UART0_RX: A78.137 (UART0_RXD), J8.1 (Pin_1), U10.1, U10.10 (NC)
- new net SOC_UART0_TX: A78.139 (UART0_TXD), J10.1 (Pin_1), U12.1, U12.10 (NC)
- new net SOC_UART1_RX: A78.141 (UART1_RXD), J8.2 (Pin_2), U10.2, U10.9 (NC)
- new net SOC_UART1_TX: A78.143 (UART1_TXD), J10.2 (Pin_2), U12.2, U12.9 (NC)
- new net SOC_UART2_RX: A78.140 (UART2_RXD), J8.3 (Pin_3), U10.4, U10.7 (NC)
- new net SOC_UART2_TX: A78.138 (UART2_TXD), J10.3 (Pin_3), U12.4, U12.7 (NC)
- new net SUSCLK_WIFI: A78.131 (SUSCLK)
- new net TMDS_CK+: C23.2, J3.10 (CK+), R16.2, U2.4, U2.7 (NC)
- new net TMDS_CK-: C24.2, J3.12 (CK-), R17.2, U2.5, U2.6 (NC)
- new net TMDS_D0+: C21.2, J3.7 (D0+), R13.2, U2.1, U2.10 (NC)
- new net TMDS_D0-: C22.2, J3.9 (D0-), R14.2, U2.2, U2.9 (NC)
- new net TMDS_D1+: C19.2, J3.4 (D1+), R9.2, U1.4, U1.7 (NC)
- new net TMDS_D1-: C20.2, J3.6 (D1-), R10.2, U1.5, U1.6 (NC)
- new net TMDS_D2+: C17.2, J3.1 (D2+), R7.2, U1.1, U1.10 (NC)
- new net TMDS_D2-: C18.2, J3.3 (D2-), R8.2, U1.2, U1.9 (NC)
- new net USB3_SSRX_N: J79.5 (SSRX-), U3.1, U3.10 (NC)
- new net USB3_SSRX_P: J79.6 (SSRX+), U3.2, U3.9 (NC)
- new net USB3_SSTX_N: C26.1
- new net USB3_SSTX_P: C27.1
- new net USB4_SSRX_N: J80.5 (SSRX-), U5.1, U5.10 (NC)
- new net USB4_SSRX_P: J80.6 (SSRX+), U5.2, U5.9 (NC)
- new net USB4_SSTX_N: C28.1
- new net USB4_SSTX_P: C29.1
- new net USB_2_P1+: A78.69 (USB2_P1+), D8.2 (A2), J80.3 (D+)
- new net USB_2_P1-: A78.67 (USB2_P1-), D78.2 (A2), J80.2 (D-)
- new net USB_2_P2+: A78.75 (USB2_P2+), D79.2 (A2), J79.3 (D+)
- new net USB_2_P2-: A78.73 (USB2_P2-), D80.2 (A2), J79.2 (D-)
- new net USB_2_P3+: A78.81 (USB2_P3+), J82.2 (Pin_2), U78.4, U78.7 (NC)
- new net USB_2_P3-: A78.79 (USB2_P3-), J82.3 (Pin_3), U78.5, U78.6 (NC)
- new net USB_2_P5+: A78.111 (USB2_P5+), J81.A6 (D+), J81.B6 (D+), U4.1, U4.10 (NC)
- new net USB_2_P5-: A78.109 (USB2_P5-), J81.A7 (D-), J81.B7 (D-), U4.2, U4.9 (NC)
- new net USB_2_P7+: A78.76 (USB2_P7+)
- new net USB_2_P7-: A78.78 (USB2_P7-)
- new net VDC: A78.250 (VIN), A78.251 (VIN), A78.252 (VIN), A78.253 (VIN), A78.254 (VIN), A78.255 (VIN), A78.256 (VIN), A78.257 (VIN), A78.258 (VIN), A78.259 (VIN), A78.260 (VIN)
- new net VPullup: R2.2
- new net ~{PEWAKE}: A78.103 (~{WAKE})
- new net ~{PWR_SW}: A78.1 (~{PWRBTN})
- new net ~{RST_SW}: A78.3 (~{RSTBTN})
- no-connect marks 3 -> 116
Other:
- removed sheet Fan_Temp
- removed sheet GPIO
- removed sheet Gigabit Ethernet
- removed sheet HDMI
- removed sheet LattePanda Module
- removed sheet M.2 E&M Key
- removed sheet PCIe x4
- removed sheet PSU
- removed sheet USB2.0&USB3.0
- note added: "DDI/TCP functions are defined by the BIOS source code, Cannot be changed in BIOS settings. Before starting design, you should choose one of the available BIOS configurations on: https://github.com/LattePandaTeam/LattePanda-Mu The default functions are defined as follows: - DDIA: eDP 1.4b (the 40Pin connector on the Mu) - DDIB: HDMI 2.0 - TCP0: HDMI 2.0 - TCP1: USB TypeC (need external PD controll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"
- note added: "HDMI"
- note added: "HPD pin of unused DDI/TCP port needs to be pulled down"
- note added: "HSIO functions are defined by the BIOS source code, Cannot be changed in BIOS settings. Before starting design, you should choose one of the available BIOS configurations on: https://github.com/LattePandaTeam/LattePanda-Mu Or contact techsupport for custom your BIOS The default functions are defined as follows: - HSIO0: USB3.2 10Gbps - HSIO1: USB3.2 10Gbps - HSIO2: PCIe 3.0 x1 - HSIO3: PCIe 3.0 x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"
- note added: "I2C has internal resistors too"
- note added: "Lattepanda Mu"
- note added: "Sleeping State Signal - SLS_S0: - S0 (Working): HIGH - S3 (Slpeeping): LOW - S4 (Hibernation): LOW - S5 (Soft Off): LOW - SLS_S3: - S0 (Working): HIGH - S3 (Slpeeping): HIGH - S4 (Hibernation): LOW - S5 (Soft Off): LOW"
- note added: "USB"
- note added: "USB2_P6 is reserved for TypeC PD Controller ONLY"
- note added: "but before there was no gnd"
- note added: "fanless"
- note added: "should be fine"
- note added: "the 4 hsio B would usually be used for pci x4 but we won't use it"
- note added: "they have internal pull up resistors"
- note added: "usb 3 seperated"
- note added: "~{CLKREQ} is reserved for PCIe ASPM L1s Unless the device clearly supports it, pull it down to enhance compatibility"
- note removed: "REFCLK can be exchange the polarity"
- moved on the sheet: FID1, FID2, H1, H2, H3, H4

Commit message: done redrawing schematic
Parts:
- added C49, C50, C55, C56: 220nF/50V, A_HDJ_Library:C_0402_1005Metric, symbol Device:C_Small
- added C51, C53, C78, C80: 10uF/10V, A_HDJ_Library:C_0402_1005Metric, symbol Device:C
- added C52, C54, C70, C71, C79, C81, C82, C84: 100nF/50V, A_HDJ_Library:C_0402_1005Metric, symbol Device:C
- added C64, C65, C67, C68, C74, C75, C76, C77, C82, C83, C85, C87: 22uF/10V, A_HDJ_Library:C_0603_1608Metric, symbol Device:C
- added C66: 1uF/16V, A_HDJ_Library:C_0402_1005Metric, symbol Device:C
- added C72, C73: 12pF/50V, Capacitor_SMD:C_0402_1005Metric, symbol Device:C
- added D15, D16, D17: SS54, A_HDJ_Library:D_SMA, symbol Device:D_Schottky
- added D21: ESD5V0B03, A_HDJ_Library:D_0402_1005Metric, symbol Diode:ESD9B5.0ST5G
- added D22, D9: LED_G, A_HDJ_Library:LED_0603_1608Metric, symbol Device:LED
- added D24: 3V3 Izt=5mA, A_HDJ_Library:D_SOD-323, symbol Device:D_Schottky
- added J15: Bus_M.2_Socket_M, A_HDJ_Library:PCIe_M.2_Connectors_P=0.5mm_H=4.2mm_KeyM, symbol Connector:Bus_M.2_Socket_M
- added J16: Bus_M.2_Socket_E, A_HDJ_Library:PCIe_M.2_Connectors_P=0.5mm_H=4.2mm_KeyE, symbol Connector:Bus_M.2_Socket_E
- added J78, J85: Conn_01x01_Pin, Connector_Wire:SolderWire-1sqmm_1x01_D1.4mm_OD2.7mm, symbol Connector:Conn_01x01_Pin
- added J83: Conn_01x02_Pin, Connector_PinHeader_2.54mm:PinHeader_1x02_P2.54mm_Vertical, symbol Connector:Conn_01x02_Pin
- added JP1: Jumper_3_Bridged12, A_HDJ_Library:PinHeader_1x03_P2.54mm_Vertical, symbol Jumper:Jumper_3_Bridged12
- added L1, L2: 2.2uH/4.3A, A_HDJ_Library:L_Sunlord_SWPA4020S, symbol Device:L
- added Q8: 2N7002, A_HDJ_Library:SOT-23, symbol Transistor_FET:2N7002
- added R27, R29, R33: 0R/1%, A_HDJ_Library:R_0402_1005Metric, symbol Device:R
- added R28: 0R/1%, Resistor_SMD:R_0402_1005Metric, symbol Device:R
- added R30, R52, R53: 2.2K/1%, A_HDJ_Library:R_0402_1005Metric, symbol Device:R
- added R34, R35, R49, R58: 10K/1%, A_HDJ_Library:R_0402_1005Metric, symbol Device:R
- added R46, R48: 100R/1%, A_HDJ_Library:R_0402_1005Metric, symbol Device:R
- added R47: 1K/1%, A_HDJ_Library:R_0402_1005Metric, symbol Device:R
- added R50: 10K/1%, Resistor_SMD:R_0402_1005Metric, symbol Device:R
- added R51: 100K/1%, A_HDJ_Library:R_0402_1005Metric, symbol Device:R
- added R57: 75K/1%, A_HDJ_Library:R_0402_1005Metric, symbol Device:R
- added R59: 21.5K/1%, A_HDJ_Library:R_0402_1005Metric, symbol Device:R
- added R60: 4.7K/1%, A_HDJ_Library:R_0402_1005Metric, symbol Device:R
- added TP13, TP2, TP5, TP6: TestPoint, A_HDJ_Library:TestPoint_Pad_D1.5mm, symbol Connector:TestPoint
- added U15, U16: SY8253ADC, A_HDJ_Library:TSOT-23-6, symbol Regulator_Switching:LM2734X
Connections:
- net +3V3: now also C51.2, C52.2, C53.2, C54.2, C73.1, C75.2, C77.2, C78.2, C79.2, C80.2, C81.2, C84.1, C85.2, C87.2, J15.12 (3.3V), J15.14 (3.3V), J15.16 (3.3V), J15.18 (3.3V), J15.2 (3.3V), J15.4 (3.3V), J15.70 (3.3V), J15.72 (3.3V), J15.74 (3.3V), J16.2 (3.3V), J16.4 (3.3V), J16.72 (3.3V), J16.74 (3.3V), L2.2, R30.2, R34.2, R35.1, R50.2, R52.2, R59.2, TP6.1
- net +5V: now also C72.1, C74.2, C76.2, C82.1, C82.2, C83.2, L1.2, R57.2, TP5.1
- net GND: now also C51.1, C52.1, C53.1, C54.1, C64.1, C65.1, C66.2, C67.1, C68.1, C74.1, C75.1, C76.1, C77.1, C78.1, C79.1, C80.1, C81.1, C82.1, C82.2, C83.1, C84.2, C85.1, C87.1, D21.1 (A1), D24.2 (A), J83.1 (Pin_1), J85.1 (Pin_1), Q8.2 (S), R27.2, R28.2, R49.1, R51.1, R58.1, R60.1, U15.2 (GND), U16.2 (GND)
- net SLS_S3: now also JP1.3 (B)
- net USB_2_P7+: now also J16.3 (USB_D+)
- net USB_2_P7-: now also J16.5 (USB_D-)
- net VPullup: now also D24.1 (K), R53.2, TP13.1
- net ~{PLT_RST}: now also J15.50 (~{PERST})
- net ~{PWR_LED}/~{PSON}: now also JP1.1 (A), R47.1
- net ~{PWR_SW}: now also R48.2
- net VDC renamed +12V
- net +12V: now also C64.2, C65.2, C67.2, C68.2, D15.1 (K), D16.1 (K), D17.1 (K), R53.1, U15.5 (VIN), U16.5 (VIN)
- new net: C72.2, R57.1, R58.2, U15.3 (FB)
- new net: C66.1, D21.2 (A2), J83.2 (Pin_2), R48.1, R50.1
- new net: J16.54 (~{W_DISABLE2}), R35.2
- new net: C71.2, U16.1 (BOOST)
- new net: C73.2, R59.1, R60.2, U16.3 (FB)
- new net: C71.1, L2.1, U16.6 (SW)
- new net: D9.2 (A), R30.1
- new net: D15.2 (A), D16.2 (A), D17.2 (A), J78.1 (Pin_1)
- new net: Q8.1 (G), R47.2, R49.2
- new net: C70.1, L1.1, U15.6 (SW)
- new net: C70.2, U15.1 (BOOST)
- new net: D9.1 (K), J15.10 (DAS/~{DSS}/~{LED1})
- new net: J16.1 (GND), J16.18 (GND), J16.33 (GND), J16.39 (GND), J16.45 (GND), J16.51 (GND), J16.57 (GND), J16.63 (GND), J16.69 (GND), J16.7 (GND), J16.75 (GND), J16.MP1, J16.MP2
- new net: C55.2, J16.35 (PETp0)
- new net: C56.2, J16.37 (PETn0)
- new net: J16.50 (SUSCLK), R33.1
- new net: J16.56 (~{W_DISABLE1}), R34.1
- new net: J15.38 (DEVSLP), TP2.1
- new net: JP1.2 (C), R46.1
- new net: D22.1 (K), Q8.3 (D)
- new net: D22.2 (A), R52.1
- new net: J15.1 (GND), J15.15 (GND), J15.21 (GND), J15.27 (GND), J15.3 (GND), J15.33 (GND), J15.39 (GND), J15.45 (GND), J15.51 (GND), J15.57 (GND), J15.71 (GND), J15.73 (GND), J15.75 (GND), J15.9 (GND), J15.MP1, J15.MP2
- new net: J15.68 (SUSCLK), R29.1
- new net: J15.69 (PEDET), R28.1
- new net CON_PCIE_TX_1+: C49.2, J15.49 (PETp0/SATA-A+)
- new net CON_PCIE_TX_1-: C50.2, J15.47 (PETn0/SATA-A-)
- new net PCIE_RX_0+: J16.41 (PERp0)
- new net PCIE_RX_0-: J16.43 (PERn0)
- new net PCIE_RX_1+: J15.43 (PERp0/SATA-B-)
- new net PCIE_RX_1-: J15.41 (PERn0/SATA-B+)
- new net PCIE_TX_0+: C55.1
- new net PCIE_TX_0-: C56.1
- new net PCIE_TX_1+: C49.1
- new net PCIE_TX_1-: C50.1
- new net PWR_EN: R46.2, R51.2, U15.4 (EN), U16.4 (EN)
- new net REFCLKE+: J16.47 (REFCLKp0)
- new net REFCLKE-: J16.49 (REFCLKn0)
- new net REFCLKM+: J15.55 (REFCLKp)
- new net REFCLKM-: J15.53 (REFCLKn)
- new net SUSCLK: R29.2, R33.2
- new net ~{CLKREQM}: J15.52 (~{CLKREQ}), R27.1
- new net ~{WAKE}: J15.54 (~{PEWAKE})
- no-connect marks 116 -> 166
Other:
- note added: "12v in"
- note added: "32.768kHz clock (for low power mode)"
- note added: "GPIO"
- note added: "M.2 E Key"
- note added: "M.2 M Key"
- note added: "M.2 connectors"
- note added: "Power"
- moved on the sheet: J10, J11, J12, J13, J14, J7, J8, J9, U10, U11, U12, U9
